File: breadboard-power-supply.kicad_pcb (KiCad board)
At the start: 2 copper layers, 53 x 30 mm, 27 parts, among them J1 PJ-002A, J2 PJ-002A, J3 TSW-102-07-F-S, J4 TSW-102-07-F-S, J5 TSW-102-07-F-S, J6 TSW-102-07-F-S, SW1 EG1271, SW2 EG2315, SW3 EG2315, U1 LM317M

Commit message: export gerbers and BOM
Other:
- board text added: "2024-10-02"
- board text removed: "2024-09-29"
Changed lines of the file:
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@@
 	(title_block
 		(title "Breadboard Power Supply")
-		(date "2024-09-29")
+		(date "2024-10-02")
 		(comment 2 "PROTOTYPE")
 		(comment 3 "2024")
@@
 			(outputformat 1)
 			(mirror no)
-			(drillshape 1)
+			(drillshape 0)
 			(scaleselection 1)
-			(outputdirectory "")
+			(outputdirectory "exports/gerbers/")
 		)
 	)
@@
 		(layer "Edge.Cuts")
 	)
-	(gr_text "2024-09-29"
+	(gr_text "2024-10-02"
 		(at 126.5 91 0)
 		(layer "B.SilkS")

Commit message: cleaned up files and scrubbed meta data
Parts:
- removed kibuzzard-66F9CAB2: G***, lib_fp:kibuzzard-66F9CAB2
- removed kibuzzard-66F9CABE: G***, lib_fp:kibuzzard-66F9CABE
- removed kibuzzard-66F9CB19: G***, lib_fp:kibuzzard-66F9CB19
- removed kibuzzard-66F9CB3C: G***, lib_fp:kibuzzard-66F9CB3C
- removed kibuzzard-66F9CB51: G***, lib_fp:kibuzzard-66F9CB51
- removed kibuzzard-66F9CBA3: G***, lib_fp:kibuzzard-66F9CBA3
- removed kibuzzard-66F9DAEC: G***, kibuzzard-66F9DAEC
- removed kibuzzard-66F9DAF8: G***, kibuzzard-66F9DAF8
- added REF***: OSHW-Logo2_7.3x6mm_SilkScreen, Symbols:OSHW-Logo2_7.3x6mm_SilkScreen, B.Cu at (126.5, 104.0)
- added kibuzzard-66FD9C27: G***, kibuzzard-66FD9C27, F.Cu at (122.9, 91.5)
- added kibuzzard-66FD9C35: G***, kibuzzard-66FD9C35, F.Cu at (118.8, 91.5)
- added kibuzzard-66FD9C43: G***, kibuzzard-66FD9C43, F.Cu at (114.7, 91.5)
- added kibuzzard-66FD9CA2: G***, kibuzzard-66FD9CA2, F.Cu at (138.8, 91.5)
- added kibuzzard-66FD9CB0: G***, kibuzzard-66FD9CB0, F.Cu at (134.2, 91.5)
- added kibuzzard-66FD9CBB: G***, kibuzzard-66FD9CBB, F.Cu at (129.6, 91.5)
- added kibuzzard-66FD9D64: G***, kibuzzard-66FD9D64, F.Cu at (113.7, 109.1)
- added kibuzzard-66FD9D69: G***, kibuzzard-66FD9D69, F.Cu at (117.8, 109.1)
- moved R3 1.84 mm to (117.7, 101.6)
- moved R2 1.82 mm to (113.9, 101.6)
- moved SW3 1.82 mm to (134.2, 97.0)
- moved SW2 1.82 mm to (118.8, 97.0)
- moved C1 1.80 mm to (121.7, 103.8)
- moved C2 1.80 mm to (131.7, 110.8)
- moved C3 1.80 mm to (135.5, 104.0)
- moved D1 1.80 mm to (124.5, 112.8)
- moved D2 1.80 mm to (132.5, 105.8)
- moved D3 1.80 mm to (124.5, 116.8)
- moved R1 1.80 mm to (135.5, 107.5)
- moved SW1 1.80 mm to (116.0, 105.3)
- moved U1 1.80 mm to (126.5, 105.8)
- renumbered D4 to D3, R5 to R3
Routing:
- net VCC1: track 78.8 -> 76.9 mm
- net Net-(J1-Pad1): track 14.8 -> 16.4 mm
- net VCC2: track 34.2 -> 32.7 mm
- net Net-(J2-Pad1): track 16.7 -> 15.4 mm
- net /ADJ: track 22.7 -> 21.8 mm
